Commit message: Remove ft sensor

File: iiwa_description/urdf/iiwa.gazebo.xacro (robot description, xacro)
@@ -5,12 +5,4 @@
     <gazebo reference="${robot_name}_joint_7">
       <provideFeedback>true</provideFeedback>
-    </gazebo>
-    <!-- The ft_sensor plugin -->
-    <gazebo>
-      <plugin name="ft_sensor" filename="libgazebo_ros_ft_sensor.so">
-        <updateRate>50.0</updateRate>
-        <topicName>/${robot_name}/state/CartesianWrench</topicName>
-        <jointName>${robot_name}_joint_7</jointName>
-      </plugin>
     </gazebo>
     <!-- Load Gazebo lib and set the robot namespace -->

File: ultrasound_probe_description/urdf/ultrasound_probe.urdf.xacro (robot description, xacro)
@@ -15,12 +15,4 @@
   <xacro:property name="camera_mass" value="0.072" />
   <xacro:property name="PI" value="3.14159265359" />
-  <!-- Force-torque sensor properties -->
-  <xacro:property name="ft_sensor_mass" value="0.120" />
-  <xacro:property name="ft_sensor_radius" value="0.03" />
-  <xacro:property name="ft_sensor_thickness" value="0.015" />
-  <xacro:property name="ft_sensor_ixx"
-                  value="${(1.0/12.0) * ft_sensor_mass * (3 * ft_sensor_radius * ft_sensor_radius + ft_sensor_thickness * ft_sensor_thickness)}" />
-  <xacro:property name="ft_sensor_izz"
-                  value="${0.5 * ft_sensor_mass * ft_sensor_radius * ft_sensor_radius}" />
   <!-- Fix to world -->
   <link name="world"/>
@@ -29,26 +21,9 @@
     <origin xyz="0 0 0" rpy="0 0 0" />
   </xacro:iiwa7>
-  <!--  Joint between the tip of the iiwa7 and the force-torque sensor -->
-  <!-- Use revolute with zero limits to enable F/T sensor plugin -->
-  <joint name="ft_sensor_joint" type="revolute">
-    <parent link="iiwa_link_ee" />
-    <child link="ft_sensor_link" />
-    <origin xyz="0 0 0" rpy="0 0 0" />
-    <axis xyz="0 0 1"/>
-    <limit lower="0" upper="0" effort="0" velocity="0"/>
-  </joint>
-  <!-- Merged F/T sensor + probe into single rigid body for force transmission -->
-  <link name="ft_sensor_link">
-    <!-- F/T sensor visual (small disk) -->
+  <!--  Ultrasound probe attached directly to robot end-effector -->
+  <link name="probe_link">
+    <!-- Probe visual -->
     <visual>
-      <origin xyz="0 0 0" rpy="0 0 0"/>
-      <geometry>
-        <cylinder length="${ft_sensor_thickness}" radius="${ft_sensor_radius}"/>
-      </geometry>
-      <material name="Grey"/>
-    </visual>
-    <!-- Probe visual (offset to account for sensor thickness) -->
-    <visual>
-      <origin xyz="0 0 ${ft_sensor_thickness/2 - 0.107}" rpy="0 0 0"/>
+      <origin xyz="0 0 -0.107" rpy="0 0 0"/>
       <geometry>
         <mesh filename="package://ultrasound_probe_description/meshes/visual/iiwa_ultrasound_probe.dae"/>
@@ -56,15 +31,15 @@
       <material name="Grey"/>
     </visual>
-    <!-- Collision for entire assembly (use probe mesh for contact) -->
+    <!-- Collision for probe -->
     <collision>
-      <origin xyz="0 0 ${ft_sensor_thickness/2 - 0.107}" rpy="0 0 0"/>
+      <origin xyz="0 0 -0.107" rpy="0 0 0"/>
       <geometry>
         <mesh filename="package://ultrasound_probe_description/meshes/collision/iiwa_ultrasound_probe.dae"/>
       </geometry>
     </collision>
-    <!-- Combined inertia (sensor + probe mass) -->
+    <!-- Probe inertia -->
     <inertial>
-      <origin xyz="0 0 ${ft_sensor_thickness/2 + 0.15}" rpy="0 0 0"/>
-      <mass value="${ft_sensor_mass + probe_mass}"/>
+      <origin xyz="0 0 0.15" rpy="0 0 0"/>
+      <mass value="${probe_mass}"/>
       <inertia ixx="0.002" ixy="0" ixz="0"
                iyy="0.002" iyz="0"
@@ -72,9 +47,15 @@
     </inertial>
   </link>
-  <!--  TCP frame at probe tip (relative to sensor link) -->
+  <!-- Joint attaching probe to robot end-effector -->
+  <joint name="probe_joint" type="fixed">
+    <parent link="iiwa_link_ee" />
+    <child link="probe_link" />
+    <origin xyz="0 0 0" rpy="0 0 0" />
+  </joint>
+  <!--  TCP frame at probe tip -->
   <joint name="probe_ee_joint" type="fixed">
-    <parent link="ft_sensor_link" />
+    <parent link="probe_link" />
     <child link="probe_link_ee" />
-    <origin xyz="0 0 ${ft_sensor_thickness/2 + probe_length}" rpy="0 0 0" />
+    <origin xyz="0 0 ${probe_length}" rpy="0 0 0" />
   </joint>
   <!--  The TCP frame -->
@@ -93,40 +74,10 @@
     </collision>
   </link>
-  <!-- Transmission for the force-torque sensor joint to expose it to ros_control -->
-  <transmission name="ft_sensor_joint_transmission">
-    <type>transmission_interface/SimpleTransmission</type>
-    <actuator name="ft_sensor_actuator">
-      <mechanicalReduction>1.0</mechanicalReduction>
-    </actuator>
-    <joint name="ft_sensor_joint">
-      <hardwareInterface>hardware_interface/PositionJointInterface</hardwareInterface>
-    </joint>
-  </transmission>
-  <!-- Gazebo contact sensor for probe collision detection and force measurement -->
-  <gazebo reference="ft_sensor_link">
-    <sensor name="probe_contact_sensor" type="contact">
-      <updateRate>100.0</updateRate>
-      <contact>
-        <collision>ft_sensor_link_collision</collision>
-      </contact>
-      <plugin name="probe_contact_plugin" filename="libgazebo_ros_bumper.so">
-        <bumperTopicName>/$(arg robot_name)/ft_sensor/wrench</bumperTopicName>
-        <frameName>ft_sensor_link</frameName>
-      </plugin>
-    </sensor>
-    <!-- Add surface properties for better contact simulation -->
-    <mu1>0.5</mu1>
-    <mu2>0.5</mu2>
-    <kp>5000.0</kp>
-    <kd>100.0</kd>
-    <minDepth>0.001</minDepth>
-  </gazebo>
   <!-- Wrist-mounted RGB-D Camera -->
-  <!-- Joint to mount camera on the side of the sensor/probe assembly -->
+  <!-- Joint to mount camera on the side of the probe assembly -->
   <joint name="wrist_camera_joint" type="fixed">
-    <parent link="ft_sensor_link" />
+    <parent link="probe_link" />
     <child link="wrist_camera_link" />
-    <!-- Adjust Z offset to account for sensor thickness -->
-    <origin xyz="0.07 0.07 ${ft_sensor_thickness/2 + 0.0725}" rpy="0 ${-PI/2} -0.75" />
+    <origin xyz="0.07 0.07 0.0725" rpy="0 ${-PI/2} -0.75" />
   </joint>
   <link name="wrist_camera_link">
